File: main_board_v2/_autosave-main_board_v2.kicad_sch (KiCad schematic)
At the start: 66 parts, among them J1 Raspberry_Pi_4, U2 Pico, U3 Pico, U4 4N35

Commit message: Work it seams
Parts:
- renumbered Servo8 to Servo10, Servo10 to Servo11, Servo3 to Servo2, Servo5 to Servo3, Servo7 to Servo4, Servo9 to Servo5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
