File: main_board_v2/main_board_v2.kicad_sch (KiCad schematic)
At the start: 66 parts, among them J1 Raspberry_Pi_4, U2 Pico, U3 Pico, U4 4N35

Commit message: Added plug for raspberry switches and corrected all DRCs
Parts:
- removed Servo11, Servo2: 1x3_PinHeader, Connector_PinHeader_2.54mm:PinHeader_1x03_P2.54mm_Vertical, symbol Connector:Conn_01x03_Pin
- added Servo5, Servo8: 1x3_PinHeader, Connector_PinHeader_2.54mm:PinHeader_1x03_P2.54mm_Vertical, symbol Connector:Conn_01x03_Pin
- added Switches1: Conn_01x06_Pin, Connector_JST:JST_PH_B6B-PH-K_1x06_P2.00mm_Vertical, symbol Connector:Conn_01x06_Pin
- renumbered Servo8 to Servo10, Servo10 to Servo11, Servo3 to Servo2, Servo5 to Servo3, U4 to U1, expansion to expansion1
Connections:
- net +3.3V: now also Switches1.2 (Pin_2)
- net +5VP: now also Servo5.2 (Pin_2)
- net +7.5V: now also Servo8.2 (Pin_2)
- net GND: now also Servo5.1 (Pin_1), Servo8.1 (Pin_1), Switches1.1 (Pin_1)
- net servo1: now also Servo2.3 (Pin_3)
- net servo10: now also Servo11.3 (Pin_3)
- net servo2: now also Servo3.3 (Pin_3); no longer Servo2.3 (Pin_3)
- net servo4: now also Servo5.3 (Pin_3); no longer Servo3.3 (Pin_3)
- net servo7: now also Servo8.3 (Pin_3); no longer Servo10.3 (Pin_3)
- net servo9: now also Servo10.3 (Pin_3); no longer Servo11.3 (Pin_3)
- net at J1.19 (MOSI0/GPIO10): now also Switches1.4 (Pin_4)
- net at J1.23 (SCLK0/GPIO11): now also Switches1.3 (Pin_3)
- net at J1.26 (~{CE1}/GPIO7): now also Switches1.5 (Pin_5)
- net at J1.31 (GCLK2/GPIO6): now also Switches1.6 (Pin_6)
