Commit message: Changed dimensions of lidar and camera resolution.

File: src/ezbot_descr_simul/description/camera.xacro (robot description, xacro)
@@ -37,6 +37,6 @@
                 <image>
                     <format>R8G8B8</format>
-                    <width>640</width>
-                    <height>480</height>
+                    <width>1280</width>
+                    <height>1280</height>
                 </image>
                 <clip>

File: src/ezbot_descr_simul/description/lidar.xacro (robot description, xacro)
@@ -9,5 +9,5 @@
         <visual>
             <geometry>
-                <cylinder radius="0.05" length="0.04"/>
+                <cylinder radius="0.02" length="0.04"/>
             </geometry>
             <material name="black"/>
@@ -22,5 +22,5 @@
         <collision>
             <geometry>
-                <cylinder radius="0.05" length="0.04"/>
+                <cylinder radius="0.02" length="0.04"/>
             </geometry>
         </collision>
@@ -33,5 +33,5 @@
         <sensor name="laser" type="ray">
             <pose> 0.055 0 0.03 0 0 0 </pose>
-            <visualize>false</visualize>
+            <visualize>true</visualize>
             <update_rate>10</update_rate>
             <ray>
