Commit message: Changed lidar frame name

File: src/ezbot_descr_simul/description/lidar.xacro (robot description, xacro)
@@ -3,8 +3,8 @@
     <joint name="laser_joint" type="fixed">
         <parent link="chassis"/>
-        <child link="laser_frame"/>
+        <child link="base_laser"/>
         <origin xyz="0.055 0 0.41" rpy="0 0 0"/>
     </joint>
-    <link name="laser_frame">
+    <link name="base_laser">
         <visual>
             <geometry>
@@ -29,5 +29,5 @@
         </xacro:inertial_cylinder>
     </link>
-    <gazebo reference="laser_frame">
+    <gazebo reference="base_laser">
         <material>Gazebo/Black</material>
         <sensor name="laser" type="ray">
@@ -53,5 +53,5 @@
                 </ros>
                 <output_type>sensor_msgs/LaserScan</output_type>
-                <frame_name>laser_frame</frame_name>
+                <frame_name>base_laser</frame_name>
             </plugin>
         </sensor>
