Commit message: robot description changes

File: src/ezbot_descr_simul/description/robot.urdf.xacro (robot description, xacro)
@@ -2,4 +2,6 @@
 <robot xmlns:xacro="http://www.ros.org/wiki/xacro"  name="robot">
     <xacro:include filename="robot_core.xacro" />
+    <xacro:include filename="lidar.xacro"/>
     <xacro:include filename="gazebo_control.xacro" />
+    <xacro:include filename="camera.xacro" />
 </robot>

File: src/ezbot_descr_simul/description/robot_core.xacro (robot description, xacro)
@@ -25,20 +25,21 @@
         <origin xyz="-0.1 0 0"/>
     </joint>
+    <!--z=0.06-->
     <link name="chassis">
         <visual>
-            <origin xyz="0.055 0 0.03"/>
-            <geometry>
-                <box size="0.11 0.11 0.06"/>
+            <origin xyz="0.055 0 0.175"/>
+            <geometry>
+                <box size="0.11 0.11 0.35"/>
             </geometry>
             <material name="orange"/>
         </visual>
         <collision>
-            <origin xyz="0.055 0 0.03"/>
-            <geometry>
-                <box size="0.11 0.11 0.06"/>
-            </geometry>
-        </collision>
-        <xacro:inertial_box mass="0.5" x="0.11" y="0.11" z="0.06">
-            <origin xyz="0.055 0 0.03" rpy="0 0 0"/>
+            <origin xyz="0.055 0 0.175"/>
+            <geometry>
+                <box size="0.11 0.11 0.35"/>
+            </geometry>
+        </collision>
+        <xacro:inertial_box mass="0.5" x="0.11" y="0.11" z="0.35">
+            <origin xyz="0.055 0 0.175" rpy="0 0 0"/>
         </xacro:inertial_box>
     </link>

Commit message: tag aruco on the robot

File: src/ezbot_descr_simul/description/robot.urdf.xacro (robot description, xacro)
@@ -5,3 +5,4 @@
     <xacro:include filename="gazebo_control.xacro" />
     <xacro:include filename="camera.xacro" />
+    <xacro:include filename="imu.xacro" />
 </robot>

File: src/ezbot_descr_simul/description/robot_core.xacro (robot description, xacro)
@@ -70,6 +70,14 @@
         </xacro:inertial_box>
     </link>
-    <gazebo reference="bloc_aruco">
-        <material>aruco/material</material>
+    <gazebo reference="bloc_aruco" link="">
+        <visual>
+        <material>
+            <script>
+                <uri>$(find ezbot_descr_simul)/media/materials/scripts</uri>
+                <uri>$(find ezbot_descr_simul)/media/materials/textures</uri>
+                <name>arucoMat</name>
+            </script>
+        </material>
+        </visual>
     </gazebo>
     <!--bloc avant-->
