Commit message: updated scale

File: src/ezbot_descr_simul/description/robot_core.xacro (robot description, xacro)
@@ -27,18 +27,18 @@
     <link name="chassis">
         <visual>
-            <origin xyz="0.55 0 0.3"/>
-            <geometry>
-                <box size="1.1 1.1 0.6"/>
+            <origin xyz="0.055 0 0.03"/>
+            <geometry>
+                <box size="0.11 0.11 0.06"/>
             </geometry>
             <material name="orange"/>
         </visual>
         <collision>
-            <origin xyz="0.55 0 0.3"/>
-            <geometry>
-                <box size="1.1 1.1 0.6"/>
-            </geometry>
-        </collision>
-        <xacro:inertial_box mass="0.5" x="1.1" y="1.1" z="0.6">
-            <origin xyz="0.55 0 0.3" rpy="0 0 0"/>
+            <origin xyz="0.055 0 0.03"/>
+            <geometry>
+                <box size="0.11 0.11 0.06"/>
+            </geometry>
+        </collision>
+        <xacro:inertial_box mass="0.5" x="0.11" y="0.11" z="0.06">
+            <origin xyz="0.055 0 0.03" rpy="0 0 0"/>
         </xacro:inertial_box>
     </link>
@@ -50,22 +50,22 @@
         <parent link="chassis"/>
         <child link="bloc_avant"/>
-        <origin xyz="1.1 0 0"/>
+        <origin xyz="0.11 0 0"/>
     </joint>
     <link name="bloc_avant">
         <visual>
-            <origin xyz="0.4 0 0.3"/>
-            <geometry>
-                <box size="0.8 0.8 0.6"/>
+            <origin xyz="0.04 0 0.03"/>
+            <geometry>
+                <box size="0.08 0.08 0.06"/>
             </geometry>
             <material name="white"/>
         </visual>
         <collision>
-            <origin xyz="0.4 0 0.3"/>
-            <geometry>
-                <box size="0.8 0.8 0.6"/>
-            </geometry>
-        </collision>
-        <xacro:inertial_box mass="0.5" x="0.8" y="0.8" z="0.6">
-            <origin xyz="0.4 0 0.3" rpy="0 0 0"/>
+            <origin xyz="0.04 0 0.03"/>
+            <geometry>
+                <box size="0.08 0.08 0.06"/>
+            </geometry>
+        </collision>
+        <xacro:inertial_box mass="0.5" x="0.08" y="0.08" z="0.06">
+            <origin xyz="0.04 0 0.03" rpy="0 0 0"/>
         </xacro:inertial_box>
     </link>
@@ -77,22 +77,22 @@
         <parent link="chassis"/>
         <child link="bloc_arriere"/>
-        <origin xyz="-0.8 0 0"/>
+        <origin xyz="-0.08 0 0"/>
     </joint>
     <link name="bloc_arriere">
         <visual>
-            <origin xyz="0.4 0 0.3"/>
-            <geometry>
-                <box size="0.8 0.8 0.6"/>
+            <origin xyz="0.04 0 0.03"/>
+            <geometry>
+                <box size="0.08 0.08 0.06"/>
             </geometry>
             <material name="black"/>
         </visual>
         <collision>
-            <origin xyz="0.4 0 0.3"/>
-            <geometry>
-                <box size="0.8 0.8 0.6"/>
-            </geometry>
-        </collision>
-        <xacro:inertial_box mass="0.5" x="0.8" y="0.8" z="0.6">
-            <origin xyz="0.4 0 0.3" rpy="0 0 0"/>
+            <origin xyz="0.04 0 0.03"/>
+            <geometry>
+                <box size="0.08 0.08 0.06"/>
+            </geometry>
+        </collision>
+        <xacro:inertial_box mass="0.05" x="0.08" y="0.08" z="0.06">
+            <origin xyz="0.04 0 0.03" rpy="0 0 0"/>
         </xacro:inertial_box>
     </link>
@@ -104,22 +104,22 @@
         <parent link="chassis"/>
         <child link="bloc_gauche"/>
-        <origin xyz="0.15 0.95 0"/>
+        <origin xyz="0.015 0.095 0"/>
     </joint>
     <link name="bloc_gauche">
         <visual>
-            <origin xyz="0.4 0 0.3"/>
-            <geometry>
-                <box size="0.8 0.8 0.6"/>
+            <origin xyz="0.04 0 0.03"/>
+            <geometry>
+                <box size="0.08 0.08 0.06"/>
             </geometry>
             <material name="black"/>
         </visual>
         <collision>
-            <origin xyz="0.4 0 0.3"/>
-            <geometry>
-                <box size="0.8 0.8 0.6"/>
-            </geometry>
-        </collision>
-        <xacro:inertial_box mass="0.5" x="0.8" y="0.8" z="0.6">
-            <origin xyz="0.4 0 0.3" rpy="0 0 0"/>
+            <origin xyz="0.04 0 0.03"/>
+            <geometry>
+                <box size="0.08 0.08 0.06"/>
+            </geometry>
+        </collision>
+        <xacro:inertial_box mass="0.5" x="0.08" y="0.08" z="0.06">
+            <origin xyz="0.04 0 0.03" rpy="0 0 0"/>
         </xacro:inertial_box>
     </link>
@@ -131,22 +131,22 @@
         <parent link="chassis"/>
         <child link="bloc_droit"/>
-        <origin xyz="0.15 -0.95 0"/>
+        <origin xyz="0.015 -0.095 0"/>
     </joint>
     <link name="bloc_droit">
         <visual>
-            <origin xyz="0.4 0 0.3"/>
-            <geometry>
-                <box size="0.8 0.8 0.6"/>
+            <origin xyz="0.04 0 0.03"/>
+            <geometry>
+                <box size="0.08 0.08 0.06"/>
             </geometry>
             <material name="black"/>
         </visual>
         <collision>
-            <origin xyz="0.4 0 0.3"/>
-            <geometry>
-                <box size="0.8 0.8 0.6"/>
-            </geometry>
-        </collision>
-        <xacro:inertial_box mass="0.5" x="0.8" y="0.8" z="0.6">
-            <origin xyz="0.4 0 0.3" rpy="0 0 0"/>
+            <origin xyz="0.04 0 0.03"/>
+            <geometry>
+                <box size="0.08 0.08 0.06"/>
+            </geometry>
+        </collision>
+        <xacro:inertial_box mass="0.5" x="0.08" y="0.08" z="0.06">
+            <origin xyz="0.04 0 0.03" rpy="0 0 0"/>
         </xacro:inertial_box>
     </link>
@@ -158,5 +158,5 @@
         <parent link="bloc_droit"/>
         <child link="roue_droite"/>
-        <origin xyz="0.4 -0.5 0.2" rpy="-${pi/2} 0 0"/>
+        <origin xyz="0.04 -0.05 0.02" rpy="-${pi/2} 0 0"/>
         <axis xyz="0 0 1"/>
     </joint>
@@ -165,13 +165,13 @@
             <material name="blue"/>
             <geometry>
-                <cylinder radius="0.3" length="0.2"/>
-            </geometry>
-        </visual>
-        <collision>
-            <geometry>
-                <cylinder radius="0.3" length="0.2"/>
-            </geometry>
-        </collision>
-        <xacro:inertial_cylinder mass="0.1" radius="0.3" length="0.2">
+                <cylinder radius="0.03" length="0.02"/>
+            </geometry>
+        </visual>
+        <collision>
+            <geometry>
+                <cylinder radius="0.03" length="0.02"/>
+            </geometry>
+        </collision>
+        <xacro:inertial_cylinder mass="0.1" radius="0.03" length="0.02">
             <origin xyz="0 0 0" rpy="0 0 0"/>
         </xacro:inertial_cylinder>
@@ -179,5 +179,4 @@
     <gazebo reference="roue_droite">
         <material>Gazebo/Blue</material>
-        <!--Have friction only along the way it rotates-->
         <fdir1>1 0 0</fdir1>
         <mu1>1.0</mu1>
@@ -188,5 +187,5 @@
         <parent link="bloc_gauche"/>
         <child link="roue_gauche"/>
-        <origin xyz="0.4 0.5 0.2" rpy="-${pi/2} 0 0"/>
+        <origin xyz="0.04 0.05 0.02" rpy="-${pi/2} 0 0"/>
         <axis xyz="0 0 1"/>
     </joint>
@@ -195,19 +194,18 @@
             <material name="blue"/>
             <geometry>
-                <cylinder radius="0.3" length="0.2"/>
-            </geometry>
-        </visual>
-        <collision>
-            <geometry>
-                <cylinder radius="0.3" length="0.2"/>
-            </geometry>
-        </collision>
-        <xacro:inertial_cylinder mass="0.1" radius="0.3" length="0.2">
+                <cylinder radius="0.03" length="0.02"/>
+            </geometry>
+        </visual>
+        <collision>
+            <geometry>
+                <cylinder radius="0.03" length="0.02"/>
+            </geometry>
+        </collision>
+        <xacro:inertial_cylinder mass="0.1" radius="0.03" length="0.02">
             <origin xyz="0 0 0" rpy="0 0 0"/>
         </xacro:inertial_cylinder>
     </link>
     <gazebo reference="roue_gauche">
-        <material>Gazebo/White</material>
-        <!--Have friction only along the way it rotates-->
+        <material>Gazebo/Blue</material>
         <fdir1>1 0 0</fdir1>
         <mu1>1.0</mu1>
@@ -218,5 +216,5 @@
         <parent link="bloc_avant"/>
         <child link="roue_avant"/>
-        <origin xyz="0.9 0 0.2" rpy="0 ${pi/2} 0"/>
+        <origin xyz="0.09 0 0.02" rpy="0 ${pi/2} 0"/>
         <axis xyz="0 0 1"/>
     </joint>
@@ -225,13 +223,13 @@
             <material name="blue"/>
             <geometry>
-                <cylinder radius="0.3" length="0.2"/>
-            </geometry>
-        </visual>
-        <collision>
-            <geometry>
-                <cylinder radius="0.3" length="0.2"/>
-            </geometry>
-        </collision>
-        <xacro:inertial_cylinder mass="0.1" radius="0.3" length="0.2">
+                <cylinder radius="0.03" length="0.02"/>
+            </geometry>
+        </visual>
+        <collision>
+            <geometry>
+                <cylinder radius="0.03" length="0.02"/>
+            </geometry>
+        </collision>
+        <xacro:inertial_cylinder mass="0.1" radius="0.03" length="0.02">
             <origin xyz="0 0 0" rpy="0 0 0"/>
         </xacro:inertial_cylinder>
@@ -247,5 +245,5 @@
         <parent link="bloc_arriere"/>
         <child link="roue_arriere"/>
-        <origin xyz="-0.1 0 0.2" rpy="0 ${pi/2} 0"/>
+        <origin xyz="-0.01 0 0.02" rpy="0 ${pi/2} 0"/>
         <axis xyz="0 0 1"/>
     </joint>
@@ -254,13 +252,13 @@
             <material name="blue"/>
             <geometry>
-                <cylinder radius="0.3" length="0.2"/>
-            </geometry>
-        </visual>
-        <collision>
-            <geometry>
-                <cylinder radius="0.3" length="0.2"/>
-            </geometry>
-        </collision>
-        <xacro:inertial_cylinder mass="0.1" radius="0.3" length="0.2">
+                <cylinder radius="0.03" length="0.02"/>
+            </geometry>
+        </visual>
+        <collision>
+            <geometry>
+                <cylinder radius="0.03" length="0.02"/>
+            </geometry>
+        </collision>
+        <xacro:inertial_cylinder mass="0.1" radius="0.03" length="0.02">
             <origin xyz="0 0 0" rpy="0 0 0"/>
         </xacro:inertial_cylinder>

Commit message: Changed color of one of the wheels

File: src/ezbot_descr_simul/description/robot_core.xacro (robot description, xacro)
@@ -208,5 +208,5 @@
     </link>
     <gazebo reference="roue_gauche">
-        <material>Gazebo/White</material>
+        <material>Gazebo/Blue</material>
         <!--Have friction only along the way it rotates-->
         <fdir1>1 0 0</fdir1>

Commit message: added an aruco marker on top of the robot

File: src/ezbot_descr_simul/description/robot_core.xacro (robot description, xacro)
@@ -47,4 +47,30 @@
         <material>Gazebo/Orange</material>
     </gazebo>
+    <!--bloc aruco-->
+    <joint name= "bloc_aruco_joint" type="fixed">
+        <parent link="chassis"/>
+        <child link="bloc_aruco"/>
+        <origin xyz="0.055 0 0"/>
+    </joint>
+    <link name="bloc_aruco">
+        <visual>
+            <origin xyz="0 0 0.47"/>
+            <geometry>
+                <box size="0.11 0.11 0.001"/>
+            </geometry>
+        </visual>
+        <collision>
+            <origin xyz="0 0 0.47"/>
+            <geometry>
+                <box size="0.11 0.11 0.001"/>
+            </geometry>
+        </collision>
+        <xacro:inertial_box mass="0.5" x="0.11" y="0.11" z="0.001">
+            <origin xyz="0 0 0.47" rpy="0 0 0"/>
+        </xacro:inertial_box>
+    </link>
+    <gazebo reference="bloc_aruco">
+        <material>aruco/material</material>
+    </gazebo>
     <!--bloc avant-->
     <joint name= "bloc_avant_joint" type="fixed">

Commit message: Added min_depth tag to (almost) eliminate the robot from drifting

File: src/ezbot_descr_simul/description/robot_core.xacro (robot description, xacro)
@@ -217,4 +217,13 @@
         <mu1>0.9</mu1>
         <mu2>0.1</mu2>
+        <collision>
+            <surface>
+                <contact>
+                <ode>
+                    <min_depth>0.01</min_depth>
+                </ode>
+                </contact>
+            </surface>
+        </collision>
     </gazebo>
     <!--roue gauche-->
@@ -246,4 +255,13 @@
         <mu1>0.9</mu1>
         <mu2>0.1</mu2>
+        <collision>
+            <surface>
+                <contact>
+                <ode>
+                    <min_depth>0.01</min_depth>
+                </ode>
+                </contact>
+            </surface>
+        </collision>
     </gazebo>
     <!--roue avant-->
@@ -275,4 +293,13 @@
         <mu1>0.9</mu1>
         <mu2>0.1</mu2>
+        <collision>
+            <surface>
+                <contact>
+                <ode>
+                    <min_depth>0.01</min_depth>
+                </ode>
+                </contact>
+            </surface>
+        </collision>
     </gazebo>
     <!--roue arriere-->
@@ -304,4 +331,13 @@
         <mu1>0.9</mu1>
         <mu2>0.1</mu2>
+        <collision>
+            <surface>
+                <contact>
+                <ode>
+                    <min_depth>0.01</min_depth>
+                </ode>
+                </contact>
+            </surface>
+        </collision>
     </gazebo>
 </robot>

Commit message: removed unused omnidirectional controller

File: src/ezbot_descr_simul/description/robot_core.xacro (robot description, xacro)
@@ -213,4 +213,43 @@
     </link>
     <gazebo reference="roue_droite">
+        <material>Gazebo/Blue</material>
+        <fdir1>1 0 0</fdir1>
+        <mu1>0.9</mu1>
+        <mu2>0.1</mu2>
+        <collision>
+            <surface>
+                <contact>
+                <ode>
+                    <max_vel>0</max_vel>clear
+                    <min_depth>0.02</min_depth>
+                </ode>
+                </contact>
+            </surface>
+        </collision>
+    </gazebo>
+    <!--roue gauche-->
+    <joint name= "roue_gauche_joint" type="continuous">
+        <parent link="bloc_gauche"/>
+        <child link="roue_gauche"/>
+        <origin xyz="0.04 0.05 0.02" rpy="-${pi/2} 0 0"/>
+        <axis xyz="0 0 1"/>
+    </joint>
+    <link name='roue_gauche'>
+        <visual>
+            <material name="blue"/>
+            <geometry>
+                <cylinder radius="0.03" length="0.02"/>
+            </geometry>
+        </visual>
+        <collision>
+            <geometry>
+                <cylinder radius="0.03" length="0.02"/>
+            </geometry>
+        </collision>
+        <xacro:inertial_cylinder mass="0.1" radius="0.03" length="0.02">
+            <origin xyz="0 0 0" rpy="0 0 0"/>
+        </xacro:inertial_cylinder>
+    </link>
+    <gazebo reference="roue_gauche">
         <material>Gazebo/Blue</material>
         <fdir1>1 0 0</fdir1>
@@ -228,12 +267,12 @@
         </collision>
     </gazebo>
-    <!--roue gauche-->
-    <joint name= "roue_gauche_joint" type="continuous">
-        <parent link="bloc_gauche"/>
-        <child link="roue_gauche"/>
-        <origin xyz="0.04 0.05 0.02" rpy="-${pi/2} 0 0"/>
+    <!--roue avant-->
+    <joint name= "roue_avant_joint" type="continuous">
+        <parent link="bloc_avant"/>
+        <child link="roue_avant"/>
+        <origin xyz="0.09 0 0.02" rpy="0 ${pi/2} 0"/>
         <axis xyz="0 0 1"/>
     </joint>
-    <link name='roue_gauche'>
+    <link name='roue_avant'>
         <visual>
             <material name="blue"/>
@@ -251,5 +290,5 @@
         </xacro:inertial_cylinder>
     </link>
-    <gazebo reference="roue_gauche">
+    <gazebo reference="roue_avant">
         <material>Gazebo/Blue</material>
         <fdir1>1 0 0</fdir1>
@@ -267,12 +306,12 @@
         </collision>
     </gazebo>
-    <!--roue avant-->
-    <joint name= "roue_avant_joint" type="continuous">
-        <parent link="bloc_avant"/>
-        <child link="roue_avant"/>
-        <origin xyz="0.09 0 0.02" rpy="0 ${pi/2} 0"/>
+    <!--roue arriere-->
+    <joint name= "roue_arriere_joint" type="continuous">
+        <parent link="bloc_arriere"/>
+        <child link="roue_arriere"/>
+        <origin xyz="-0.01 0 0.02" rpy="0 ${pi/2} 0"/>
         <axis xyz="0 0 1"/>
     </joint>
-    <link name='roue_avant'>
+    <link name='roue_arriere'>
         <visual>
             <material name="blue"/>
@@ -290,5 +329,5 @@
         </xacro:inertial_cylinder>
     </link>
-    <gazebo reference="roue_avant">
+    <gazebo reference="roue_arriere">
         <material>Gazebo/Blue</material>
         <fdir1>1 0 0</fdir1>
@@ -306,43 +345,4 @@
         </collision>
     </gazebo>
-    <!--roue arriere-->
-    <joint name= "roue_arriere_joint" type="continuous">
-        <parent link="bloc_arriere"/>
-        <child link="roue_arriere"/>
-        <origin xyz="-0.01 0 0.02" rpy="0 ${pi/2} 0"/>
-        <axis xyz="0 0 1"/>
-    </joint>
-    <link name='roue_arriere'>
-        <visual>
-            <material name="blue"/>
-            <geometry>
-                <cylinder radius="0.03" length="0.02"/>
-            </geometry>
-        </visual>
-        <collision>
-            <geometry>
-                <cylinder radius="0.03" length="0.02"/>
-            </geometry>
-        </collision>
-        <xacro:inertial_cylinder mass="0.1" radius="0.03" length="0.02">
-            <origin xyz="0 0 0" rpy="0 0 0"/>
-        </xacro:inertial_cylinder>
-    </link>
-    <gazebo reference="roue_arriere">
-        <material>Gazebo/Blue</material>
-        <fdir1>1 0 0</fdir1>
-        <mu1>0.9</mu1>
-        <mu2>0.1</mu2>
-        <collision>
-            <surface>
-                <contact>
-                <ode>
-                    <max_vel>0</max_vel>
-                    <min_depth>0.02</min_depth>
-                </ode>
-                </contact>
-            </surface>
-        </collision>
-    </gazebo>
     <link name="renverseur_de_panneaux">
         <visual>
