Commit message: added marker detection for the second camera

File: src/ezbot_static_camera/description/camera_static.xacro (robot description, xacro)
@@ -6,5 +6,5 @@
         <origin xyz="0 0 0" rpy="0 1.57 0"/>
     </joint>
-    <link name="camera_link">
+    <link name="camera_link" type="fixed">
         <visual>
             <geometry>
@@ -12,12 +12,8 @@
             </geometry>
         </visual>
-        <gazebo>
-            <static>true</static>
-            <gravity>false</gravity>
-        </gazebo>
     </link>
-    <gazebo reference="camera_link">
+    <gazebo reference="camera_link" type="fixed">
         <material>Gazebo/Black</material>
-        <gravity>false</gravity>
+        <static>true</static>
         <sensor name="camera2" type="camera">
             <pose> 0 0 0 0 0 0 </pose>
@@ -25,5 +21,5 @@
             <update_rate>10</update_rate>
             <camera>
-                <horizontal_fov>1.089</horizontal_fov>
+                <horizontal_fov>2</horizontal_fov>
                 <image>
                     <format>R8G8B8</format>

File: src/ezbot_static_camera/description/robot_core.xacro (robot description, xacro)
@@ -5,13 +5,15 @@
         <color rgba="1 0.3 0.1 1"/>
     </material>
-    <link name="base_link">
-    </link>
+    <link name="base_link"></link>
+    <gazebo>
+        <static>true</static>
+    </gazebo>
     <!--Chassis-->
     <joint name= "chassis_joint" type="fixed">
         <parent link="base_link"/>
         <child link="chassis"/>
-        <origin xyz="0 -0.35 3"/>
+        <origin xyz="0 0 0"/>
     </joint>
-    <link name="chassis">
+    <link name="chassis" type="fixed">
         <visual>
             <origin xyz="0 0 0"/>
@@ -31,6 +33,7 @@
         </xacro:inertial_box>
     </link>
-    <gazebo reference="chassis">
-    <gravity>false</gravity>
+    <gazebo reference="chassis" type="fixed">
+        <static>true</static>
+        <gravity>false</gravity>
         <material>Gazebo/Orange</material>
     </gazebo>
