Commit message: ros2_control seem to be working, testing the communication with Pico

File: src/ezbot_robot/description/robot.urdf.xacro (robot description, xacro)
@@ -3,5 +3,8 @@
     <xacro:include filename="robot_core.xacro" />
     <xacro:include filename="lidar.xacro"/>
-    <xacro:include filename="gazebo_control.xacro" />
+    <xacro:include filename="ros2_control.xacro" />
+    <!--
+        <xacro:include filename="gazebo_control.xacro" />
+    -->
     <xacro:include filename="camera.xacro" />
     <xacro:include filename="imu.xacro" />

File: src/ezbot_robot/description/ros2_control.xacro (robot description, xacro)
@@ -1,5 +1,5 @@
 <?xml version="1.0"?>
 <robot xmlns:xacro="http://www.ros.org/wiki/xacro">
-    <ros2_control name="ros2_control_wheel_joint" type="system">
+    <ros2_control name="hellothere" type="system">
         <hardware>
             <plugin>omnidrive_rppico/OmniDriveRpPicoHardware</plugin>
@@ -8,41 +8,41 @@
             <param name="back_wheel_name">roue_arriere_joint</param>
             <param name="right_wheel_name">roue_droite_joint</param>
-            <param name="loop_rate">30</param>
-            <param name="device">/dev/pts/9</param>
+            <param name="loop_rate">30.0</param>
+            <param name="device">/dev/pts/7</param>
             <param name="baudrate">115200</param>
             <param name="timeout_ms">10000</param>
             <param name="enc_counts_per_rev">3600</param>
         </hardware>
-        <joint name="roue_avant_joint1">
+        <joint name="roue_avant_joint">
             <command_interface name="velocity">
                 <param name="min">-10</param>
                 <param name="max">10</param>
             </command_interface>
+            <state_interface name="position"/>
             <state_interface name="velocity"/>
-            <state_interface name="position"/>
         </joint>
-        <joint name="roue_gauche_joint2">
+        <joint name="roue_gauche_joint">
             <command_interface name="velocity">
                 <param name="min">-10</param>
                 <param name="max">10</param>
             </command_interface>
+            <state_interface name="position"/>
             <state_interface name="velocity"/>
-            <state_interface name="position"/>
         </joint>
-        <joint name="roue_arriere_joint3">
+        <joint name="roue_arriere_joint">
             <command_interface name="velocity">
                 <param name="min">-10</param>
                 <param name="max">10</param>
             </command_interface>
+            <state_interface name="position"/>
             <state_interface name="velocity"/>
-            <state_interface name="position"/>
         </joint>
-        <joint name="roue_droite_joint4">
+        <joint name="roue_droite_joint">
             <command_interface name="velocity">
                 <param name="min">-10</param>
                 <param name="max">10</param>
             </command_interface>
+            <state_interface name="position"/>
             <state_interface name="velocity"/>
-            <state_interface name="position"/>
         </joint>
     </ros2_control>
