Commit message: Reverted the removed controller and fixed some bugs
This controller is based on @mateusmenezes95 3 wheel omnidirectional controller.

File: src/ezbot_robot/description/robot_core.xacro (robot description, xacro)
@@ -213,43 +213,4 @@
     </link>
     <gazebo reference="roue_droite">
-        <material>Gazebo/Blue</material>
-        <fdir1>1 0 0</fdir1>
-        <mu1>0.9</mu1>
-        <mu2>0.1</mu2>
-        <collision>
-            <surface>
-                <contact>
-                <ode>
-                    <max_vel>0</max_vel>clear
-                    <min_depth>0.02</min_depth>
-                </ode>
-                </contact>
-            </surface>
-        </collision>
-    </gazebo>
-    <!--roue gauche-->
-    <joint name= "roue_gauche_joint" type="continuous">
-        <parent link="bloc_gauche"/>
-        <child link="roue_gauche"/>
-        <origin xyz="0.04 0.05 0.02" rpy="-${pi/2} 0 0"/>
-        <axis xyz="0 0 1"/>
-    </joint>
-    <link name='roue_gauche'>
-        <visual>
-            <material name="blue"/>
-            <geometry>
-                <cylinder radius="0.03" length="0.02"/>
-            </geometry>
-        </visual>
-        <collision>
-            <geometry>
-                <cylinder radius="0.03" length="0.02"/>
-            </geometry>
-        </collision>
-        <xacro:inertial_cylinder mass="0.1" radius="0.03" length="0.02">
-            <origin xyz="0 0 0" rpy="0 0 0"/>
-        </xacro:inertial_cylinder>
-    </link>
-    <gazebo reference="roue_gauche">
         <material>Gazebo/Blue</material>
         <fdir1>1 0 0</fdir1>
@@ -267,12 +228,12 @@
         </collision>
     </gazebo>
-    <!--roue avant-->
-    <joint name= "roue_avant_joint" type="continuous">
-        <parent link="bloc_avant"/>
-        <child link="roue_avant"/>
-        <origin xyz="0.09 0 0.02" rpy="0 ${pi/2} 0"/>
+    <!--roue gauche-->
+    <joint name= "roue_gauche_joint" type="continuous">
+        <parent link="bloc_gauche"/>
+        <child link="roue_gauche"/>
+        <origin xyz="0.04 0.05 0.02" rpy="-${pi/2} 0 0"/>
         <axis xyz="0 0 1"/>
     </joint>
-    <link name='roue_avant'>
+    <link name='roue_gauche'>
         <visual>
             <material name="blue"/>
@@ -290,5 +251,5 @@
         </xacro:inertial_cylinder>
     </link>
-    <gazebo reference="roue_avant">
+    <gazebo reference="roue_gauche">
         <material>Gazebo/Blue</material>
         <fdir1>1 0 0</fdir1>
@@ -306,12 +267,12 @@
         </collision>
     </gazebo>
-    <!--roue arriere-->
-    <joint name= "roue_arriere_joint" type="continuous">
-        <parent link="bloc_arriere"/>
-        <child link="roue_arriere"/>
-        <origin xyz="-0.01 0 0.02" rpy="0 ${pi/2} 0"/>
+    <!--roue avant-->
+    <joint name= "roue_avant_joint" type="continuous">
+        <parent link="bloc_avant"/>
+        <child link="roue_avant"/>
+        <origin xyz="0.09 0 0.02" rpy="0 ${pi/2} 0"/>
         <axis xyz="0 0 1"/>
     </joint>
-    <link name='roue_arriere'>
+    <link name='roue_avant'>
         <visual>
             <material name="blue"/>
@@ -329,5 +290,5 @@
         </xacro:inertial_cylinder>
     </link>
-    <gazebo reference="roue_arriere">
+    <gazebo reference="roue_avant">
         <material>Gazebo/Blue</material>
         <fdir1>1 0 0</fdir1>
@@ -345,4 +306,43 @@
         </collision>
     </gazebo>
+    <!--roue arriere-->
+    <joint name= "roue_arriere_joint" type="continuous">
+        <parent link="bloc_arriere"/>
+        <child link="roue_arriere"/>
+        <origin xyz="-0.01 0 0.02" rpy="0 ${pi/2} 0"/>
+        <axis xyz="0 0 1"/>
+    </joint>
+    <link name='roue_arriere'>
+        <visual>
+            <material name="blue"/>
+            <geometry>
+                <cylinder radius="0.03" length="0.02"/>
+            </geometry>
+        </visual>
+        <collision>
+            <geometry>
+                <cylinder radius="0.03" length="0.02"/>
+            </geometry>
+        </collision>
+        <xacro:inertial_cylinder mass="0.1" radius="0.03" length="0.02">
+            <origin xyz="0 0 0" rpy="0 0 0"/>
+        </xacro:inertial_cylinder>
+    </link>
+    <gazebo reference="roue_arriere">
+        <material>Gazebo/Blue</material>
+        <fdir1>1 0 0</fdir1>
+        <mu1>0.9</mu1>
+        <mu2>0.1</mu2>
+        <collision>
+            <surface>
+                <contact>
+                <ode>
+                    <max_vel>0</max_vel>
+                    <min_depth>0.02</min_depth>
+                </ode>
+                </contact>
+            </surface>
+        </collision>
+    </gazebo>
     <link name="renverseur_de_panneaux">
         <visual>

File: src/ezbot_robot/description/ros2_control.xacro (robot description, xacro)
@@ -9,5 +9,5 @@
             <param name="right_wheel_name">roue_droite_joint</param>
             <param name="loop_rate">30</param>
-            <param name="device">/dev/ttyAMA1</param>
+            <param name="device">/dev/pts/11</param>
             <param name="baudrate">115200</param>
             <param name="timeout_ms">10000</param>

Commit message: Added base_footprint link

File: src/ezbot_robot/description/robot_core.xacro (robot description, xacro)
@@ -25,4 +25,11 @@
         <origin xyz="-0.1 0 0"/>
     </joint>
+    <joint name= "base_footprint_joint" type="fixed">
+        <parent link="base_link"/>
+        <child link="base_footprint"/>
+        <origin xyz="0 0 0"/>
+    </joint>
+    <link name="base_footprint">
+    </link>
     <!--z=0.06-->
     <link name="chassis">

Commit message: changed who is the parent and who is the child

File: src/ezbot_robot/description/robot_core.xacro (robot description, xacro)
@@ -25,11 +25,11 @@
         <origin xyz="-0.1 0 0"/>
     </joint>
+    <link name="base_footprint">
+    </link>
     <joint name= "base_footprint_joint" type="fixed">
-        <parent link="base_link"/>
-        <child link="base_footprint"/>
+        <parent link="base_footprint"/>
+        <child link="base_link"/>
         <origin xyz="0 0 0"/>
     </joint>
-    <link name="base_footprint">
-    </link>
     <!--z=0.06-->
     <link name="chassis">

Commit message: Changed base_link and base foot_print relationship

File: src/ezbot_robot/description/robot_core.xacro (robot description, xacro)
@@ -28,6 +28,6 @@
     </link>
     <joint name= "base_footprint_joint" type="fixed">
-        <parent link="base_footprint"/>
-        <child link="base_link"/>
+        <parent link="base_link"/>
+        <child link="base_footprint"/>
         <origin xyz="0 0 0"/>
     </joint>

Commit message: Switched footprint to be parent

File: src/ezbot_robot/description/robot_core.xacro (robot description, xacro)
@@ -28,6 +28,6 @@
     </link>
     <joint name= "base_footprint_joint" type="fixed">
-        <parent link="base_link"/>
-        <child link="base_footprint"/>
+        <parent link="base_footprint"/>
+        <child link="base_link"/>
         <origin xyz="0 0 0"/>
     </joint>
