Commit message: Added joint ldlidar_base

File: src/ezbot_robot/description/lidar.xacro (robot description, xacro)
@@ -5,4 +5,9 @@
         <child link="base_laser"/>
         <origin xyz="0.055 0 0.41" rpy="0 0 0"/>
+    </joint>
+    <joint name="ldlidar_base" type="fixed">
+        <parent link="base_laser"/>
+        <child link="ldlidar"/>
+        <origin xyz="0 0 0" rpy="0 0 0"/>
     </joint>
     <link name="base_laser">

Commit message: changed description xacro

File: src/ezbot_robot/description/lidar.xacro (robot description, xacro)
@@ -6,9 +6,11 @@
         <origin xyz="0.055 0 0.41" rpy="0 0 0"/>
     </joint>
-    <joint name="ldlidar_base" type="fixed">
+    <joint name="ldlidar_node" type="fixed">
         <parent link="base_laser"/>
-        <child link="ldlidar"/>
+        <child link="ldlidar_base"/>
         <origin xyz="0 0 0" rpy="0 0 0"/>
     </joint>
+    <link name="ldlidar_base">
+    </link>
     <link name="base_laser">
         <visual>

Commit message: rotated joint

File: src/ezbot_robot/description/lidar.xacro (robot description, xacro)
@@ -9,5 +9,5 @@
         <parent link="base_laser"/>
         <child link="ldlidar_base"/>
-        <origin xyz="0 0 0" rpy="0 0 0"/>
+        <origin xyz="0 0 0" rpy="0 0 1.5708"/>
     </joint>
     <link name="ldlidar_base">

Commit message: wrong way

File: src/ezbot_robot/description/lidar.xacro (robot description, xacro)
@@ -9,5 +9,5 @@
         <parent link="base_laser"/>
         <child link="ldlidar_base"/>
-        <origin xyz="0 0 0" rpy="0 0 1.5708"/>
+        <origin xyz="0 0 0" rpy="0 0 -1.5708"/>
     </joint>
     <link name="ldlidar_base">

Commit message: Robot worky, lidar rotated around
around the world around the world around the world around the world around the world around the world around the world around the world

File: src/ezbot_robot/description/lidar.xacro (robot description, xacro)
@@ -9,5 +9,5 @@
         <parent link="base_laser"/>
         <child link="ldlidar_base"/>
-        <origin xyz="0 0 0" rpy="0 0 -1.5708"/>
+        <origin xyz="0 0 0" rpy="0 0 1.5708"/>
     </joint>
     <link name="ldlidar_base">

Commit message: Changed rotation of lidar yet again

File: src/ezbot_robot/description/lidar.xacro (robot description, xacro)
@@ -9,5 +9,5 @@
         <parent link="base_laser"/>
         <child link="ldlidar_base"/>
-        <origin xyz="0 0 0" rpy="0 0 1.5708"/>
+        <origin xyz="0 0 0" rpy="0 0 0"/>
     </joint>
     <link name="ldlidar_base">

Commit message: Added link to ldlidar_link in lidar.xacro

File: src/ezbot_robot/description/lidar.xacro (robot description, xacro)
@@ -12,4 +12,11 @@
     </joint>
     <link name="ldlidar_base">
+    </link>
+    <joint name="ldlidar_link_node" type="fixed">
+        <parent link="base_laser"/>
+        <child link="ldlidar_link"/>
+        <origin xyz="0 0 0" rpy="0 0 0"/>
+    </joint>
+    <link name="ldlidar_link">
     </link>
     <link name="base_laser">
